Commit message: Title: Added basic envs for Mobile Robot use-case
Body: Added a maze and empty env for a mobile robot use case using the
kobuki robot. The maze env is still going through revisions as the
training is taking too long and possibly the size of the maze is going
to be reduced. The training of the empty env is already completed and
the logs were generated for both TD3 and SAC.

Authored-by: Jose Fajardo <jmfajardod@unal.edu.co>

File: kobuki_maze/kobuki/kobuki_description/urdf/kobuki_gazebo.urdf.xacro (robot description, xacro)
@@ -160,4 +160,5 @@
       </sensor>
     </gazebo>
+    <!--
     <gazebo>
       <plugin name="kobuki_controller" filename="libgazebo_ros_kobuki.so">
@@ -177,4 +178,30 @@
       </plugin>
     </gazebo>
+    -->
+    <gazebo>
+      <plugin name="differential_drive_controller" filename="libgazebo_ros_diff_drive.so">
+        <updateRate>60</updateRate>
+        <leftJoint>wheel_left_joint</leftJoint>
+        <rightJoint>wheel_right_joint</rightJoint>
+        <wheelSeparation>0.230</wheelSeparation>
+        <wheelDiameter>0.070</wheelDiameter>
+        <wheelAcceleration>1.0</wheelAcceleration>
+        <wheelTorque>20</wheelTorque>
+        <commandTopic>cmd_vel</commandTopic>
+        <odometryTopic>odom</odometryTopic>
+        <odometryFrame>odom</odometryFrame>
+        <robotBaseFrame>base_footprint</robotBaseFrame>
+        <!-- Odometry source, 0 for ENCODER, 1 for WORLD, defaults to WORLD -->
+        <odometrySource>1</odometrySource>
+        <!-- Set to true to publish transforms for the wheel links, defaults to false -->
+        <publishWheelTF>true</publishWheelTF>
+        <!-- Set to true to publish transforms for the odometry, defaults to true -->
+        <publishOdom>true</publishOdom>
+        <!-- Set to true to publish sensor_msgs/JointState on /joint_states for the wheel joints, defaults to false -->
+        <publishWheelJointState>true</publishWheelJointState>
+        <!-- Set to true to swap right and left wheels, defaults to true -->
+        <legacyMode>false</legacyMode>
+      </plugin>
+    </gazebo>
   </xacro:macro>
 </robot>

File: kobuki_maze/kobuki_maze_rl/urdf/kobuki_lidar.gazebo.xacro (robot description, xacro)
@@ -7,5 +7,5 @@
             <pose>0 0 0 0 0 0</pose>
             <visualize>$(arg laser_visual)</visualize>
-            <update_rate>40</update_rate>
+            <update_rate>60</update_rate>
             <ray>
                 <scan>

File: kobuki_maze/kobuki_maze_rl/urdf/kobuki_lidar.urdf.xacro (robot description, xacro)
@@ -6,5 +6,5 @@
     <xacro:include filename="$(find kobuki_maze_rl)/urdf/kobuki_lidar.gazebo.xacro" />
     <joint name="camera_joint" type="fixed">
-        <origin xyz="0.08 0.0 0.12" rpy="0 0 0"/>
+        <origin xyz="0.0 0.0 0.12" rpy="0 0 0"/>
         <parent link="base_link"/>
         <child link="base_scan"/>
