Commit message: removed collision meshes of links

File: ur5_reacher/ur_description/urdf/ur5.urdf.xacro (robot description, xacro)
@@ -86,9 +86,9 @@
         </material>
       </visual>
-      <collision>
+      <!-- <collision>
         <geometry>
           <mesh filename="package://ur_description/meshes/ur5/collision/base.stl" />
         </geometry>
-      </collision>
+      </collision> -->
       <xacro:cylinder_inertial radius="0.06" length="0.05" mass="${base_mass}">
         <origin xyz="0.0 0.0 0.0" rpy="0 0 0" />
@@ -123,9 +123,9 @@
         </material>
       </visual>
-      <collision>
+      <!-- <collision>
         <geometry>
           <mesh filename="package://ur_description/meshes/ur5/collision/shoulder.stl" />
         </geometry>
-      </collision>
+      </collision> -->
       <xacro:cylinder_inertial radius="0.06" length="0.15" mass="${shoulder_mass}">
         <origin xyz="0.0 0.0 0.0" rpy="0 0 0" />
@@ -161,9 +161,9 @@
         </material>
       </visual>
-      <collision>
+      <!-- <collision>
         <geometry>
           <mesh filename="package://ur_description/meshes/ur5/collision/upperarm.stl" />
         </geometry>
-      </collision>
+      </collision> -->
       <xacro:cylinder_inertial radius="0.06" length="0.56" mass="${upper_arm_mass}">
         <origin xyz="0.0 0.0 0.28" rpy="0 0 0" />
@@ -198,9 +198,9 @@
         </material>
       </visual>
-      <collision>
+      <!-- <collision>
         <geometry>
           <mesh filename="package://ur_description/meshes/ur5/collision/forearm.stl" />
         </geometry>
-      </collision>
+      </collision> -->
       <xacro:cylinder_inertial radius="0.06" length="${-a3}" mass="${forearm_mass}">
         <origin xyz="0.0 0.0 ${-a3/2}" rpy="0 0 0" />
@@ -235,9 +235,9 @@
         </material>
       </visual>
-      <collision>
+      <!-- <collision>
         <geometry>
           <mesh filename="package://ur_description/meshes/ur5/collision/wrist1.stl" />
         </geometry>
-      </collision>
+      </collision> -->
       <xacro:cylinder_inertial radius="0.06" length="0.12" mass="${wrist_1_mass}">
         <origin xyz="0.0 ${wrist_1_length} 0.0" rpy="0 0 0" />
@@ -272,9 +272,9 @@
         </material>
       </visual>
-      <collision>
+      <!-- <collision>
         <geometry>
           <mesh filename="package://ur_description/meshes/ur5/collision/wrist2.stl" />
         </geometry>
-      </collision>
+      </collision> -->
       <xacro:cylinder_inertial radius="0.06" length="0.12" mass="${wrist_2_mass}">
         <origin xyz="0.0 0.0 ${wrist_2_length}" rpy="0 0 0" />
@@ -309,9 +309,9 @@
         </material>
       </visual>
-      <collision>
+      <!-- <collision>
         <geometry>
           <mesh filename="package://ur_description/meshes/ur5/collision/wrist3.stl" />
         </geometry>
-      </collision>
+      </collision> -->
       <xacro:cylinder_inertial radius="0.0375" length="0.0345" mass="${wrist_3_mass}">
         <origin xyz="0.0 ${wrist_3_length - 0.0345/2} 0.0" rpy="${pi/2} 0 0" />
@@ -324,10 +324,10 @@
     </joint>
     <link name="${prefix}ee_link">
-      <collision>
+      <!-- <collision>
         <geometry>
           <box size="0.01 0.01 0.01"/>
         </geometry>
         <origin rpy="0 0 0" xyz="-0.01 0 0"/>
-      </collision>
+      </collision> -->
     </link>
     <xacro:ur_arm_transmission prefix="${prefix}" hw_interface="${transmission_hw_interface}" />
